File: eps/v1/hardware/5V_voltage_regulator.kicad_sch (KiCad schematic)
At the start: 23 parts, among them U40 MP28167-A

Commit message: share footprint & symbol libraries
Parts:
- U40: symbol EPS:MP28167-A -> OSUSAT_EPS:MP28167-A
Changed lines of the file:
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@@
 	)
 	(symbol
-		(lib_id "EPS:MP28167-A")
+		(lib_id "OSUSAT_EPS:MP28167-A")
 		(at 140.97 91.44 0)
 		(unit 1)
