File: eps/v1/hardware/battery_charger.kicad_sch (KiCad schematic)
At the start: 18 parts, among them J9 Conn_01x03, Q1 NMOS, Q2 NMOS, U3 LTC4162-L

Commit message: share footprint & symbol libraries
Parts:
- U3: symbol EPS:LTC4162-L -> OSUSAT_EPS:LTC4162-L
Changed lines of the file:
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@@
 	)
 	(symbol
-		(lib_id "EPS:LTC4162-L")
+		(lib_id "OSUSAT_EPS:LTC4162-L")
 		(at 99.06 33.02 0)
 		(unit 1)
