File: eps/v1/hardware/power_path_ideal_diode.kicad_sch (KiCad schematic)
At the start: 9 parts, among them U41 LTC4415

Commit message: share footprint & symbol libraries
Parts:
- U41: symbol EPS:LTC4415 -> OSUSAT_EPS:LTC4415
Changed lines of the file:
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@@
 	)
 	(symbol
-		(lib_id "EPS:LTC4415")
+		(lib_id "OSUSAT_EPS:LTC4415")
 		(at 142.24 71.12 0)
 		(unit 1)
