File: backplane/v1/hardware/3u/backplane.kicad_sch (KiCad schematic)
At the start: 1 part, among them J1 Conn_02x20_Odd_Even

Commit message: add initial 3U design
Parts:
- added H1, H2, H3, H4, H5, H6: MountingHole, MountingHole:MountingHole_4.3mm_M4, symbol Mechanical:MountingHole
- added H10, H7, H8, H9: MountingHole_Pad, MountingHole:MountingHole_3.2mm_M3_Pad, symbol Mechanical:MountingHole_Pad
- added J10, J11, J12, J2, J3, J4, J5, J6, J7, J8, J9: Conn_02x20_Odd_Even, footprints:SFM-120-X1-XXX-D, symbol Connector_Generic:Conn_02x20_Odd_Even
- J1: footprint (none) -> footprints:SFM-120-X1-XXX-D
Connections:
- net GND: now reaches J1.1 (Pin_1)
- net GND: now also J1.19 (Pin_19), J1.2 (Pin_2), J1.20 (Pin_20), J1.22 (Pin_22), J1.39 (Pin_39), J1.40 (Pin_40), J1.LC1, J1.LC2, H10.1, H7.1, H8.1, H9.1, J10.1 (Pin_1), J10.19 (Pin_19), J10.2 (Pin_2), J10.20 (Pin_20), J10.22 (Pin_22), J10.39 (Pin_39), J10.40 (Pin_40), J10.LC1, J10.LC2, J11.1 (Pin_1), J11.19 (Pin_19), J11.2 (Pin_2), J11.20 (Pin_20), J11.22 (Pin_22), J11.39 (Pin_39), J11.40 (Pin_40), J11.LC1, J11.LC2, J12.1 (Pin_1), J12.19 (Pin_19), J12.2 (Pin_2), J12.20 (Pin_20), J12.22 (Pin_22), J12.39 (Pin_39), J12.40 (Pin_40), J12.LC1, J12.LC2, J2.1 (Pin_1), J2.19 (Pin_19), J2.2 (Pin_2), J2.20 (Pin_20), J2.22 (Pin_22), J2.39 (Pin_39), J2.40 (Pin_40), J2.LC1, J2.LC2, J3.1 (Pin_1), J3.19 (Pin_19), J3.2 (Pin_2), J3.20 (Pin_20), J3.22 (Pin_22), J3.39 (Pin_39), J3.40 (Pin_40), J3.LC1, J3.LC2, J4.1 (Pin_1), J4.19 (Pin_19), J4.2 (Pin_2), J4.20 (Pin_20), J4.22 (Pin_22), J4.39 (Pin_39), J4.40 (Pin_40), J4.LC1, J4.LC2, J5.1 (Pin_1), J5.19 (Pin_19), J5.2 (Pin_2), J5.20 (Pin_20), J5.22 (Pin_22), J5.39 (Pin_39), J5.40 (Pin_40), J5.LC1, J5.LC2, J6.1 (Pin_1), J6.19 (Pin_19), J6.2 (Pin_2), J6.20 (Pin_20), J6.22 (Pin_22), J6.39 (Pin_39), J6.40 (Pin_40), J6.LC1, J6.LC2, J7.1 (Pin_1), J7.19 (Pin_19), J7.2 (Pin_2), J7.20 (Pin_20), J7.22 (Pin_22), J7.39 (Pin_39), J7.40 (Pin_40), J7.LC1, J7.LC2, J8.1 (Pin_1), J8.19 (Pin_19), J8.2 (Pin_2), J8.20 (Pin_20), J8.22 (Pin_22), J8.39 (Pin_39), J8.40 (Pin_40), J8.LC1, J8.LC2, J9.1 (Pin_1), J9.19 (Pin_19), J9.2 (Pin_2), J9.20 (Pin_20), J9.22 (Pin_22), J9.39 (Pin_39), J9.40 (Pin_40), J9.LC1, J9.LC2
- net RAIL_4_VOUT: now reaches J1.10 (Pin_10)
- net RAIL_4_VOUT: now also J1.9 (Pin_9), J10.10 (Pin_10), J10.9 (Pin_9), J11.10 (Pin_10), J11.9 (Pin_9), J12.10 (Pin_10), J12.9 (Pin_9), J2.10 (Pin_10), J2.9 (Pin_9), J3.10 (Pin_10), J3.9 (Pin_9), J4.10 (Pin_10), J4.9 (Pin_9), J5.10 (Pin_10), J5.9 (Pin_9), J6.10 (Pin_10), J6.9 (Pin_9), J7.10 (Pin_10), J7.9 (Pin_9), J8.10 (Pin_10), J8.9 (Pin_9), J9.10 (Pin_10), J9.9 (Pin_9)
- net RAIL_5_VOUT: now reaches J1.11 (Pin_11)
- net RAIL_5_VOUT: now also J1.12 (Pin_12), J10.11 (Pin_11), J10.12 (Pin_12), J11.11 (Pin_11), J11.12 (Pin_12), J12.11 (Pin_11), J12.12 (Pin_12), J2.11 (Pin_11), J2.12 (Pin_12), J3.11 (Pin_11), J3.12 (Pin_12), J4.11 (Pin_11), J4.12 (Pin_12), J5.11 (Pin_11), J5.12 (Pin_12), J6.11 (Pin_11), J6.12 (Pin_12), J7.11 (Pin_11), J7.12 (Pin_12), J8.11 (Pin_11), J8.12 (Pin_12), J9.11 (Pin_11), J9.12 (Pin_12)
- net RAIL_6_VOUT: now reaches J1.13 (Pin_13)
- net RAIL_6_VOUT: now also J1.14 (Pin_14), J10.13 (Pin_13), J10.14 (Pin_14), J11.13 (Pin_13), J11.14 (Pin_14), J12.13 (Pin_13), J12.14 (Pin_14), J2.13 (Pin_13), J2.14 (Pin_14), J3.13 (Pin_13), J3.14 (Pin_14), J4.13 (Pin_13), J4.14 (Pin_14), J5.13 (Pin_13), J5.14 (Pin_14), J6.13 (Pin_13), J6.14 (Pin_14), J7.13 (Pin_13), J7.14 (Pin_14), J8.13 (Pin_13), J8.14 (Pin_14), J9.13 (Pin_13), J9.14 (Pin_14)
- net RAIL_7_VOUT: now reaches J1.15 (Pin_15)
- net RAIL_7_VOUT: now also J1.16 (Pin_16), J10.15 (Pin_15), J10.16 (Pin_16), J11.15 (Pin_15), J11.16 (Pin_16), J12.15 (Pin_15), J12.16 (Pin_16), J2.15 (Pin_15), J2.16 (Pin_16), J3.15 (Pin_15), J3.16 (Pin_16), J4.15 (Pin_15), J4.16 (Pin_16), J5.15 (Pin_15), J5.16 (Pin_16), J6.15 (Pin_15), J6.16 (Pin_16), J7.15 (Pin_15), J7.16 (Pin_16), J8.15 (Pin_15), J8.16 (Pin_16), J9.15 (Pin_15), J9.16 (Pin_16)
- net RAIL_8_VOUT: now reaches J1.17 (Pin_17)
- net RAIL_8_VOUT: now also J1.18 (Pin_18), J10.17 (Pin_17), J10.18 (Pin_18), J11.17 (Pin_17), J11.18 (Pin_18), J12.17 (Pin_17), J12.18 (Pin_18), J2.17 (Pin_17), J2.18 (Pin_18), J3.17 (Pin_17), J3.18 (Pin_18), J4.17 (Pin_17), J4.18 (Pin_18), J5.17 (Pin_17), J5.18 (Pin_18), J6.17 (Pin_17), J6.18 (Pin_18), J7.17 (Pin_17), J7.18 (Pin_18), J8.17 (Pin_17), J8.18 (Pin_18), J9.17 (Pin_17), J9.18 (Pin_18)
- net EPS_PGOOD: now reaches J1.21 (Pin_21)
- net EPS_PGOOD: now also J10.21 (Pin_21), J11.21 (Pin_21), J12.21 (Pin_21), J2.21 (Pin_21), J3.21 (Pin_21), J4.21 (Pin_21), J5.21 (Pin_21), J6.21 (Pin_21), J7.21 (Pin_21), J8.21 (Pin_21), J9.21 (Pin_21)
- net CAN_MAIN_P: now reaches J1.23 (Pin_23)
- net CAN_MAIN_P: now also J1.24 (Pin_24), J10.23 (Pin_23), J10.24 (Pin_24), J11.23 (Pin_23), J11.24 (Pin_24), J12.23 (Pin_23), J12.24 (Pin_24), J2.23 (Pin_23), J2.24 (Pin_24), J3.23 (Pin_23), J3.24 (Pin_24), J4.23 (Pin_23), J4.24 (Pin_24), J5.23 (Pin_23), J5.24 (Pin_24), J6.23 (Pin_23), J6.24 (Pin_24), J7.23 (Pin_23), J7.24 (Pin_24), J8.23 (Pin_23), J8.24 (Pin_24), J9.23 (Pin_23), J9.24 (Pin_24)
- net CAN_MAIN_N: now reaches J1.25 (Pin_25)
- net CAN_MAIN_N: now also J1.26 (Pin_26), J10.25 (Pin_25), J10.26 (Pin_26), J11.25 (Pin_25), J11.26 (Pin_26), J12.25 (Pin_25), J12.26 (Pin_26), J2.25 (Pin_25), J2.26 (Pin_26), J3.25 (Pin_25), J3.26 (Pin_26), J4.25 (Pin_25), J4.26 (Pin_26), J5.25 (Pin_25), J5.26 (Pin_26), J6.25 (Pin_25), J6.26 (Pin_26), J7.25 (Pin_25), J7.26 (Pin_26), J8.25 (Pin_25), J8.26 (Pin_26), J9.25 (Pin_25), J9.26 (Pin_26)
- net OBC_HEARTBEAT: now reaches J1.27 (Pin_27)
- net OBC_HEARTBEAT: now also J10.27 (Pin_27), J11.27 (Pin_27), J12.27 (Pin_27), J2.27 (Pin_27), J3.27 (Pin_27), J4.27 (Pin_27), J5.27 (Pin_27), J6.27 (Pin_27), J7.27 (Pin_27), J8.27 (Pin_27), J9.27 (Pin_27)
- net EPS_OBC_RESET: now reaches J1.28 (Pin_28)
- net EPS_OBC_RESET: now also J10.28 (Pin_28), J11.28 (Pin_28), J12.28 (Pin_28), J2.28 (Pin_28), J3.28 (Pin_28), J4.28 (Pin_28), J5.28 (Pin_28), J6.28 (Pin_28), J7.28 (Pin_28), J8.28 (Pin_28), J9.28 (Pin_28)
- net SLOT_ID0: now reaches J1.29 (Pin_29)
- net SLOT_ID0: now also J10.29 (Pin_29), J11.29 (Pin_29), J12.29 (Pin_29), J2.29 (Pin_29), J3.29 (Pin_29), J4.29 (Pin_29), J5.29 (Pin_29), J6.29 (Pin_29), J7.29 (Pin_29), J8.29 (Pin_29), J9.29 (Pin_29)
- net RAIL_1_VOUT: now reaches J1.3 (Pin_3)
- net RAIL_1_VOUT: now also J1.4 (Pin_4), J10.3 (Pin_3), J10.4 (Pin_4), J11.3 (Pin_3), J11.4 (Pin_4), J12.3 (Pin_3), J12.4 (Pin_4), J2.3 (Pin_3), J2.4 (Pin_4), J3.3 (Pin_3), J3.4 (Pin_4), J4.3 (Pin_3), J4.4 (Pin_4), J5.3 (Pin_3), J5.4 (Pin_4), J6.3 (Pin_3), J6.4 (Pin_4), J7.3 (Pin_3), J7.4 (Pin_4), J8.3 (Pin_3), J8.4 (Pin_4), J9.3 (Pin_3), J9.4 (Pin_4)
- net OBC_EPS_RESET: now reaches J1.30 (Pin_30)
- net OBC_EPS_RESET: now also J10.30 (Pin_30), J11.30 (Pin_30), J12.30 (Pin_30), J2.30 (Pin_30), J3.30 (Pin_30), J4.30 (Pin_30), J5.30 (Pin_30), J6.30 (Pin_30), J7.30 (Pin_30), J8.30 (Pin_30), J9.30 (Pin_30)
- net SLOT_ID1: now reaches J1.31 (Pin_31)
- net SLOT_ID1: now also J10.31 (Pin_31), J11.31 (Pin_31), J12.31 (Pin_31), J2.31 (Pin_31), J3.31 (Pin_31), J4.31 (Pin_31), J5.31 (Pin_31), J6.31 (Pin_31), J7.31 (Pin_31), J8.31 (Pin_31), J9.31 (Pin_31)
- net SLOT_ID2: now reaches J1.32 (Pin_32)
- net SLOT_ID2: now also J10.32 (Pin_32), J11.32 (Pin_32), J12.32 (Pin_32), J2.32 (Pin_32), J3.32 (Pin_32), J4.32 (Pin_32), J5.32 (Pin_32), J6.32 (Pin_32), J7.32 (Pin_32), J8.32 (Pin_32), J9.32 (Pin_32)
- net SPI_SCLK: now reaches J1.33 (Pin_33)
- net SPI_SCLK: now also J10.33 (Pin_33), J11.33 (Pin_33), J12.33 (Pin_33), J2.33 (Pin_33), J3.33 (Pin_33), J4.33 (Pin_33), J5.33 (Pin_33), J6.33 (Pin_33), J7.33 (Pin_33), J8.33 (Pin_33), J9.33 (Pin_33)
- net SPI_MOSI: now reaches J1.34 (Pin_34)
- net SPI_MOSI: now also J10.34 (Pin_34), J11.34 (Pin_34), J12.34 (Pin_34), J2.34 (Pin_34), J3.34 (Pin_34), J4.34 (Pin_34), J5.34 (Pin_34), J6.34 (Pin_34), J7.34 (Pin_34), J8.34 (Pin_34), J9.34 (Pin_34)
- net SPI_MISO: now reaches J1.35 (Pin_35)
- net SPI_MISO: now also J10.35 (Pin_35), J11.35 (Pin_35), J12.35 (Pin_35), J2.35 (Pin_35), J3.35 (Pin_35), J4.35 (Pin_35), J5.35 (Pin_35), J6.35 (Pin_35), J7.35 (Pin_35), J8.35 (Pin_35), J9.35 (Pin_35)
- net CAN_AUX_P: now reaches J1.36 (Pin_36)
- net CAN_AUX_P: now also J10.36 (Pin_36), J11.36 (Pin_36), J12.36 (Pin_36), J2.36 (Pin_36), J3.36 (Pin_36), J4.36 (Pin_36), J5.36 (Pin_36), J6.36 (Pin_36), J7.36 (Pin_36), J8.36 (Pin_36), J9.36 (Pin_36)
- net SPARE1: now reaches J1.37 (Pin_37)
- net SPARE1: now also J10.37 (Pin_37), J11.37 (Pin_37), J12.37 (Pin_37), J2.37 (Pin_37), J3.37 (Pin_37), J4.37 (Pin_37), J5.37 (Pin_37), J6.37 (Pin_37), J7.37 (Pin_37), J8.37 (Pin_37), J9.37 (Pin_37)
- net CAN_AUX_N: now reaches J1.38 (Pin_38)
- net CAN_AUX_N: now also J10.38 (Pin_38), J11.38 (Pin_38), J12.38 (Pin_38), J2.38 (Pin_38), J3.38 (Pin_38), J4.38 (Pin_38), J5.38 (Pin_38), J6.38 (Pin_38), J7.38 (Pin_38), J8.38 (Pin_38), J9.38 (Pin_38)
- net RAIL_2_VOUT: now reaches J1.5 (Pin_5)
- net RAIL_2_VOUT: now also J1.6 (Pin_6), J10.5 (Pin_5), J10.6 (Pin_6), J11.5 (Pin_5), J11.6 (Pin_6), J12.5 (Pin_5), J12.6 (Pin_6), J2.5 (Pin_5), J2.6 (Pin_6), J3.5 (Pin_5), J3.6 (Pin_6), J4.5 (Pin_5), J4.6 (Pin_6), J5.5 (Pin_5), J5.6 (Pin_6), J6.5 (Pin_5), J6.6 (Pin_6), J7.5 (Pin_5), J7.6 (Pin_6), J8.5 (Pin_5), J8.6 (Pin_6), J9.5 (Pin_5), J9.6 (Pin_6)
- net RAIL_3_VOUT: now reaches J1.7 (Pin_7)
- net RAIL_3_VOUT: now also J1.8 (Pin_8), J10.7 (Pin_7), J10.8 (Pin_8), J11.7 (Pin_7), J11.8 (Pin_8), J12.7 (Pin_7), J12.8 (Pin_8), J2.7 (Pin_7), J2.8 (Pin_8), J3.7 (Pin_7), J3.8 (Pin_8), J4.7 (Pin_7), J4.8 (Pin_8), J5.7 (Pin_7), J5.8 (Pin_8), J6.7 (Pin_7), J6.8 (Pin_8), J7.7 (Pin_7), J7.8 (Pin_8), J8.7 (Pin_7), J8.8 (Pin_8), J9.7 (Pin_7), J9.8 (Pin_8)
Other:
- note added: "ADCS"
- note added: "BAT"
- note added: "COMM"
- note added: "EPS"
- note added: "GENERIC"
- note added: "OBC"
- note added: "PAYLOAD"
- note added: "Recommended Stackup: JLC04161H-7628"
