File: backplane/v1/hardware/flatsat/daughterboard_connectors.kicad_sch (KiCad schematic)
At the start: 8 parts, among them J1 Conn_02x20_Odd_Even, J2 Conn_02x20_Odd_Even, J3 Conn_02x20_Odd_Even, J4 Conn_02x20_Odd_Even, J5 Conn_02x20_Odd_Even, J6 Conn_02x20_Odd_Even, J7 Conn_02x20_Odd_Even, J8 Conn_02x20_Odd_Even

Commit message: add silk & clean flatsat
Parts:
- added R1, R2, R3, R4, R5, R6, R7, R8: 20m, Resistor_SMD:R_1206_3216Metric, symbol Device:R_Small_US
- renumbered J3 to J1, J1 to J3
Connections:
- net RAIL_1_VOUT: now also R1.1; no longer J2.3 (Pin_3), J2.4 (Pin_4)
- net RAIL_2_VOUT: now also R2.1; no longer J3.5 (Pin_5), J3.6 (Pin_6)
- net RAIL_3_VOUT: now also R3.1; no longer J5.7 (Pin_7), J5.8 (Pin_8)
- net RAIL_4_VOUT: now also R4.1; no longer J6.10 (Pin_10), J6.9 (Pin_9)
- net RAIL_5_VOUT: now also R5.1; no longer J7.11 (Pin_11), J7.12 (Pin_12)
- net RAIL_6_VOUT: now also R8.1; no longer J4.13 (Pin_13), J4.14 (Pin_14)
- net RAIL_7_VOUT: now also R6.1; no longer J8.15 (Pin_15), J8.16 (Pin_16)
- net RAIL_8_VOUT: now also R7.1; no longer J1.17 (Pin_17), J1.18 (Pin_18)
- new net R1: J2.3 (Pin_3), J2.4 (Pin_4), R1.2
- new net R2: J3.5 (Pin_5), J3.6 (Pin_6), R2.2
- new net R3: J5.7 (Pin_7), J5.8 (Pin_8), R3.2
- new net R4: J6.10 (Pin_10), J6.9 (Pin_9), R4.2
- new net R5: J7.11 (Pin_11), J7.12 (Pin_12), R5.2
- new net R6: J4.13 (Pin_13), J4.14 (Pin_14), R8.2
- new net R7: J8.15 (Pin_15), J8.16 (Pin_16), R6.2
- new net R8: J1.17 (Pin_17), J1.18 (Pin_18), R7.2
