File: backplane/v1/hardware/flatsat/flatsat.kicad_pcb (KiCad board)
At the start: 4 copper layers, 464 x 286 mm, 8 parts, among them J1 Conn_02x20_Odd_Even, J2 Conn_02x20_Odd_Even, J3 Conn_02x20_Odd_Even, J4 Conn_02x20_Odd_Even, J5 Conn_02x20_Odd_Even, J6 Conn_02x20_Odd_Even, J7 Conn_02x20_Odd_Even, J8 Conn_02x20_Odd_Even

Commit message: fix connector orientation on flatsat
Parts:
- moved J1 18.5 mm to (119.8, 150.3)
- moved J2 18.5 mm to (230.8, 150.3)
- moved J3 18.5 mm to (341.8, 150.3)
- moved J4 18.5 mm to (452.8, 150.3)
- moved J5 18.5 mm to (119.8, 283.3)
- moved J6 18.5 mm to (230.8, 283.3)
- moved J7 18.5 mm to (341.8, 283.3)
- moved J8 18.5 mm to (452.8, 283.3)
Routing:
- net SPI_MOSI: track 1000.3 -> 963.3 mm
- net EPS_PGOOD: track 959.8 -> 922.9 mm
- net EPS_OBC_RESET: track 980.6 -> 943.7 mm
- net OBC_EPS_RESET: track 987.4 -> 950.5 mm
- net CAN_AUX_P: track 1015.6 -> 978.7 mm
- net SPI_SCLK: track 993.6 -> 956.8 mm
- net SPI_MISO: track 1008.3 -> 971.5 mm
- net OBC_HEARTBEAT: track 973.4 -> 936.7 mm
- net CAN_MAIN_N: track 1006.9 -> 970.6 mm
- net SPARE1: track 1023.5 -> 987.2 mm
- net CAN_AUX_N: track 1031.6 -> 995.5 mm
- net CAN_MAIN_P: track 1004.1 -> 1016.1 mm, vias 9 -> 10
- net GND: track 114.9 -> 106.9 mm, vias 26 -> 24
- net RAIL_8_VOUT: vias 30 -> 26
- added copper zone on In2.Cu, net GND

Commit message: add silk & clean flatsat
Parts:
- added G***: LOGO, LOGO, F.Cu at (166.2, 172.9)
- added R1: 20m, Resistor_SMD:R_1206_3216Metric, F.Cu at (204.2, 156.2)
- added R2: 20m, Resistor_SMD:R_1206_3216Metric, F.Cu at (318.8, 156.7)
- added R3: 20m, Resistor_SMD:R_1206_3216Metric, F.Cu at (100.2, 290.4)
- added R4: 20m, Resistor_SMD:R_1206_3216Metric, F.Cu at (214.8, 292.4)
- added R5: 20m, Resistor_SMD:R_1206_3216Metric, F.Cu at (329.3, 292.6)
- added R6: 20m, Resistor_SMD:R_1206_3216Metric, F.Cu at (447.3, 292.4)
- added R7: 20m, Resistor_SMD:R_1206_3216Metric, F.Cu at (117.8, 157.6)
- added R8: 20m, Resistor_SMD:R_1206_3216Metric, F.Cu at (443.8, 160.1)
Connections:
- J1 pad 17: RAIL_8_VOUT -> /Daughterboard Connectors/R8
- J1 pad 18: RAIL_8_VOUT -> /Daughterboard Connectors/R8
- J1 pad 31: unconnected-(J1-Pin_31-Pad31) -> GND
- J2 pad 3: RAIL_1_VOUT -> /Daughterboard Connectors/R1
- J2 pad 4: RAIL_1_VOUT -> /Daughterboard Connectors/R1
- J3 pad 31: GND -> unconnected-(J3-Pin_31-Pad31)
- J3 pad 5: RAIL_2_VOUT -> /Daughterboard Connectors/R2
- J3 pad 6: RAIL_2_VOUT -> /Daughterboard Connectors/R2
- J4 pad 13: RAIL_6_VOUT -> /Daughterboard Connectors/R6
- J4 pad 14: RAIL_6_VOUT -> /Daughterboard Connectors/R6
- J5 pad 7: RAIL_3_VOUT -> /Daughterboard Connectors/R3
- J5 pad 8: RAIL_3_VOUT -> /Daughterboard Connectors/R3
- J6 pad 10: RAIL_4_VOUT -> /Daughterboard Connectors/R4
- J6 pad 9: RAIL_4_VOUT -> /Daughterboard Connectors/R4
- J7 pad 11: RAIL_5_VOUT -> /Daughterboard Connectors/R5
- J7 pad 12: RAIL_5_VOUT -> /Daughterboard Connectors/R5
- J8 pad 15: RAIL_7_VOUT -> /Daughterboard Connectors/R7
- J8 pad 16: RAIL_7_VOUT -> /Daughterboard Connectors/R7
Routing:
- net RAIL_1_VOUT: track 174.5 -> 152.7 mm
- net /Daughterboard Connectors/R1: track 0.00 -> 19.1 mm
- net RAIL_2_VOUT: track 152.3 -> 133.2 mm
- net RAIL_3_VOUT: track 133.1 -> 116.5 mm
- net /Daughterboard Connectors/R2: track 0.00 -> 16.2 mm
- net /Daughterboard Connectors/R3: track 0.00 -> 14.3 mm
- net RAIL_4_VOUT: track 109.4 -> 95.7 mm
- net /Daughterboard Connectors/R4: track 0.00 -> 13.3 mm
- net RAIL_5_VOUT: track 90.4 -> 79.1 mm
- net /Daughterboard Connectors/R5: track 0.00 -> 11.3 mm
- net RAIL_6_VOUT: track 70.8 -> 62.0 mm
- net /Daughterboard Connectors/R6: track 0.00 -> 8.85 mm
- net RAIL_7_VOUT: track 63.4 -> 55.5 mm
- net /Daughterboard Connectors/R7: track 0.00 -> 7.29 mm
- net GND: track 106.9 -> 107.8 mm
- added copper zone on F.Cu, net /Daughterboard Connectors/R8
Other:
- board text added: "ADCS"
- board text added: "BAT"
- board text added: "COMM"
- board text added: "DOWN↓"
- board text added: "EPS"
- board text added: "GEN"
- board text added: "OBC"
- board text added: "OSUSat 2026 FlatSat v1r1"
- board text added: "PAY"
- board text added: "UP↑"

Commit message: add shunt resistors, rail injection points, and breakout
Parts:
- added J10: Conn_01x02, Connector_AMASS:AMASS_XT30UPB-F_1x02_P5.0mm_Vertical, F.Cu at (52.0, 85.8)
- added J11: Conn_01x02, Connector_AMASS:AMASS_XT30UPB-F_1x02_P5.0mm_Vertical, F.Cu at (52.0, 106.5)
- added J12: Conn_01x02, Connector_AMASS:AMASS_XT30UPB-F_1x02_P5.0mm_Vertical, F.Cu at (52.0, 127.2)
- added J13: Conn_01x02, Connector_AMASS:AMASS_XT30UPB-F_1x02_P5.0mm_Vertical, F.Cu at (52.0, 218.8)
- added J14: Conn_01x02, Connector_AMASS:AMASS_XT30UPB-F_1x02_P5.0mm_Vertical, F.Cu at (52.0, 239.5)
- added J15: Conn_01x02, Connector_AMASS:AMASS_XT30UPB-F_1x02_P5.0mm_Vertical, F.Cu at (52.0, 260.2)
- added J16: Conn_01x02, Connector_AMASS:AMASS_XT30UPB-F_1x02_P5.0mm_Vertical, F.Cu at (52.0, 281.0)
- added J17: Conn_01x11, Connector_PinHeader_2.54mm:PinHeader_1x11_P2.54mm_Vertical, F.Cu at (504.0, 327.6)
- added J9: Conn_01x02, Connector_AMASS:AMASS_XT30UPB-F_1x02_P5.0mm_Vertical, F.Cu at (52.0, 65.0)
Routing:
- net CAN_MAIN_N: track 970.6 -> 1177.1 mm, vias 9 -> 11
- net CAN_MAIN_P: track 1016.1 -> 1222.2 mm, vias 10 -> 12
- net RAIL_1_VOUT: track 152.7 -> 264.9 mm, vias 30 -> 34
- net RAIL_8_VOUT: track 0.00 -> 96.8 mm, vias 26 -> 30
- net RAIL_2_VOUT: track 133.2 -> 226.5 mm, vias 30 -> 34
- net RAIL_7_VOUT: track 55.5 -> 133.5 mm, vias 30 -> 34
- net RAIL_3_VOUT: track 116.5 -> 191.0 mm, vias 30 -> 34
- net RAIL_6_VOUT: track 62.0 -> 121.3 mm, vias 30 -> 34
- net RAIL_4_VOUT: track 95.7 -> 151.4 mm, vias 30 -> 34
- net RAIL_5_VOUT: track 79.1 -> 119.5 mm, vias 30 -> 34
- net EPS_PGOOD: track 922.9 -> 962.7 mm
- net OBC_HEARTBEAT: track 936.7 -> 973.9 mm
- net EPS_OBC_RESET: track 943.7 -> 980.2 mm
- net OBC_EPS_RESET: track 950.5 -> 986.4 mm
- net SPI_SCLK: track 956.8 -> 991.9 mm
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