File: backplane/v1/hardware/flatsat/instrumentation.kicad_sch (KiCad schematic)
At the start: 0 parts

Commit message: add shunt resistors, rail injection points, and breakout
Parts:
- added J10, J11, J12, J13, J14, J15, J16, J9: Conn_01x02, Connector_AMASS:AMASS_XT30UPB-F_1x02_P5.0mm_Vertical, symbol Connector_Generic:Conn_01x02
- added J17: Conn_01x11, Connector_PinHeader_2.54mm:PinHeader_1x11_P2.54mm_Vertical, symbol Connector_Generic:Conn_01x11
Connections:
- new net CAN_AUX_N: J17.9 (Pin_9)
- new net CAN_AUX_P: J17.8 (Pin_8)
- new net CAN_MAIN_N: J17.11 (Pin_11)
- new net CAN_MAIN_P: J17.10 (Pin_10)
- new net EPS_OBC_RESET: J17.3 (Pin_3)
- new net EPS_PGOOD: J17.1 (Pin_1)
- new net GND: J10.1 (Pin_1), J11.1 (Pin_1), J12.1 (Pin_1), J13.1 (Pin_1), J14.1 (Pin_1), J15.1 (Pin_1), J16.1 (Pin_1), J9.1 (Pin_1)
- new net OBC_EPS_RESET: J17.4 (Pin_4)
- new net OBC_HEARTBEAT: J17.2 (Pin_2)
- new net RAIL_1_VOUT: J9.2 (Pin_2)
- new net RAIL_2_VOUT: J10.2 (Pin_2)
- new net RAIL_3_VOUT: J11.2 (Pin_2)
- new net RAIL_4_VOUT: J12.2 (Pin_2)
- new net RAIL_5_VOUT: J13.2 (Pin_2)
- new net RAIL_6_VOUT: J14.2 (Pin_2)
- new net RAIL_7_VOUT: J15.2 (Pin_2)
- new net RAIL_8_VOUT: J16.2 (Pin_2)
- new net SPI_MISO: J17.7 (Pin_7)
- new net SPI_MOSI: J17.6 (Pin_6)
- new net SPI_SCLK: J17.5 (Pin_5)
