File: backplane/v1/hardware/test_board/rp2040.kicad_sch (KiCad schematic)
At the start: 23 parts, among them J3 Conn_01x02, U2 RP2040, U3 W25Q128JVS, Y1 12MHz

Commit message: add burnwire & IMU peripherals
Connections:
- net +3V3: no longer C12.1, C13.1, C14.1, C15.1, C16.1, C17.1, C18.1, C23.1, U2.1 (IOVDD), U2.10 (IOVDD), U2.22 (IOVDD), U2.33 (IOVDD), U2.42 (IOVDD), U2.43 (ADC_AVDD), U2.44 (VREG_VIN), U2.48 (USB_VDD), U2.49 (IOVDD)
- new net RAIL_1_VOUT: C12.1, C13.1, C14.1, C15.1, C16.1, C17.1, C18.1, C23.1, U2.1 (IOVDD), U2.10 (IOVDD), U2.22 (IOVDD), U2.33 (IOVDD), U2.42 (IOVDD), U2.43 (ADC_AVDD), U2.44 (VREG_VIN), U2.48 (USB_VDD), U2.49 (IOVDD)
- no-connect marks 20 -> 18
Other:
- title: (none) -> Daughterboard
Changed lines of the file:
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@@
 	(generator_version "10.0")
 	(paper "A4")
+	(title_block
+		(title "Daughterboard")
+	)
 	(rectangle
 		(start 180.34 85.09)
@@
 	)
 	(junction
-		(at 81.28 39.37)
-		(diameter 0)
-		(color 0 0 0 0)
-	)
-	(junction
 		(at 248.92 96.52)
 		(diameter 0)
@@
 	)
 	(no_connect
-		(at 68.58 149.86)
-	)
-	(no_connect
 		(at 119.38 132.08)
 	)
@@
 	)
 	(no_connect
-		(at 68.58 147.32)
-	)
-	(no_connect
 		(at 119.38 134.62)
 	)
@@
 	(wire
 		(pts
-			(xy 86.36 39.37) (xy 81.28 39.37)
+			(xy 76.2 39.37) (xy 86.36 39.37)
 		)
 		(stroke
@@
 	(wire
 		(pts
-			(xy 81.28 39.37) (xy 76.2 39.37)
-		)
-		(stroke
-			(width 0)
-			(type default)
-		)
-	)
-	(wire
-		(pts
 			(xy 96.52 54.61) (xy 96.52 73.66)
 		)
@@
 	(wire
 		(pts
-			(xy 88.9 36.83) (xy 88.9 39.37)
+			(xy 88.9 31.75) (xy 88.9 39.37)
 		)
 		(stroke
@@
 	(wire
 		(pts
-			(xy 81.28 35.56) (xy 81.28 39.37)
-		)
-		(stroke
-			(width 0)
-			(type default)
-		)
-	)
-	(wire
-		(pts
 			(xy 127 49.53) (xy 113.03 49.53)
 		)
@@
 		)
 	)
+	(wire
+		(pts
+			(xy 85.09 31.75) (xy 88.9 31.75)
+		)
+		(stroke
+			(width 0)
+			(type default)
+		)
+	)
 	(label "PI_D+"
 		(at 59.69 106.68 0)
@@
 		)
 	)
+	(hierarchical_label "RAIL_1_VOUT"
+		(shape input)
+		(at 85.09 31.75 180)
+		(effects
+			(font
+				(size 1.27 1.27)
+				(thickness 0.1588)
+			)
+			(justify right)
+		)
+	)
 	(hierarchical_label "USB_D-"
 		(shape bidirectional)
@@
 	)
 	(symbol
-		(lib_id "power:PWR_FLAG")
-		(at 81.28 35.56 0)
-		(mirror y)
-		(unit 1)
-		(body_style 1)
-		(exclude_from_sim no)
-		(in_bom yes)
-		(on_board yes)
-		(in_pos_files yes)
-		(dnp no)
-		(fields_autoplaced yes)
-		(property "Reference" "#FLG03"
-			(at 81.28 33.655 0)
-			(hide yes)
-			(show_name no)
-			(do_not_autoplace no)
-			(effects
-				(font
-					(size 1.27 1.27)
-				)
-			)
-		)
-		(property "Value" "PWR_FLAG"
-			(at 81.28 30.48 0)
-			(show_name no)
-			(do_not_autoplace no)
-			(effects
-				(font
-					(size 1.27 1.27)
-				)
-			)
-		)
-		(property "Footprint" ""
-			(at 81.28 35.56 0)
-			(hide yes)
-			(show_name no)
-			(do_not_autoplace no)
-			(effects
-				(font
-					(size 1.27 1.27)
-				)
-			)
-		)
-		(property "Datasheet" ""
-			(at 81.28 35.56 0)
-			(hide yes)
-			(show_name no)
-			(do_not_autoplace no)
-			(effects
-				(font
-					(size 1.27 1.27)
-				)
-			)
-		)
-		(property "Description" "Special symbol for telling ERC where power comes from"
-			(at 81.28 35.56 0)
-			(hide yes)
-			(show_name no)
-			(do_not_autoplace no)
-			(effects
-				(font
-					(size 1.27 1.27)
-				)
-			)
-		)
-		(pin "1"
-		)
-		(instances
-			(project "test_board"
-				(path "/b20f5a9e-495e-48d8-8648-bd5c7d9b4620/caa5ee9e-9d51-4a25-9811-e48a0e8c4a80"
-					(reference "#FLG03")
-					(unit 1)
-				)
-			)
-		)
-	)
-	(symbol
 		(lib_id "Connector_Generic:Conn_01x02")
 		(at 186.69 114.3 0)
@@
 					(unit 1)
 				)
-			)
-		)
-	)
-	(symbol
-		(lib_id "power:+3V3")
-		(at 88.9 36.83 0)
-		(unit 1)
-		(body_style 1)
-		(exclude_from_sim no)
-		(in_bom yes)
-		(on_board yes)
-		(in_pos_files yes)
-		(dnp no)
-		(fields_autoplaced yes)
-		(property "Reference" "#PWR011"
-			(at 88.9 40.64 0)
-			(hide yes)
-			(show_name no)
-			(do_not_autoplace no)
-			(effects
-				(font
-					(size 1.27 1.27)
-				)
-			)
-		)
-		(property "Value" "+3V3"
-			(at 88.9 31.75 0)
-			(show_name no)
-			(do_not_autoplace no)
-			(effects
-				(font
-					(size 1.27 1.27)
-				)
-			)
-		)
-		(property "Footprint" ""
-			(at 88.9 36.83 0)
-			(hide yes)
-			(show_name no)
-			(do_not_autoplace no)
-			(effects
-				(font
-					(size 1.27 1.27)
-				)
-			)
-		)
-		(property "Datasheet" ""
-			(at 88.9 36.83 0)
-			(hide yes)
-			(show_name no)
-			(do_not_autoplace no)
-			(effects
-				(font
-					(size 1.27 1.27)
-				)
-			)
-		)
-		(property "Description" "Power symbol creates a global label with name \"+3V3\""
-			(at 88.9 36.83 0)
-			(hide yes)
-			(show_name no)
-			(do_not_autoplace no)
-			(effects
-				(font
-					(size 1.27 1.27)
-				)
-			)
-		)
-		(pin "1"
-		)
-		(instances
-			(project "test_board"
-				(path "/b20f5a9e-495e-48d8-8648-bd5c7d9b4620/caa5ee9e-9d51-4a25-9811-e48a0e8c4a80"
-					(reference "#PWR011")
-					(unit 1)
-				)

Commit message: add ADC peripherals to test board
Connections:
- net BURNWIRE_GATE: now reaches U2.2 (GPIO0)
- net IMU_INT: now reaches U2.3 (GPIO1)
- net IMU_SCL: now reaches U2.4 (GPIO2)
- net IMU_SDA: now reaches U2.5 (GPIO3)
- no-connect marks 18 -> 16
Changed lines of the file:
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@@
-	)
-	(no_connect
-		(at 119.38 152.4)
 	)
 	(no_connect
@@
 	)
 	(no_connect
-		(at 119.38 149.86)
-	)
-	(no_connect
 		(at 68.58 154.94)
 	)
@@
 	(wire
 		(pts
+			(xy 119.38 83.82) (xy 139.7 83.82)
+		)
+		(stroke
+			(width 0)
+			(type default)
+		)
+	)
+	(wire
+		(pts
 			(xy 127 39.37) (xy 127 41.91)
 		)
@@
 	(wire
 		(pts
+			(xy 119.38 86.36) (xy 139.7 86.36)
+		)
+		(stroke
+			(width 0)
+			(type default)
+		)
+	)
+	(wire
+		(pts
 			(xy 194.31 52.07) (xy 203.2 52.07)
 		)
@@
 	(wire
 		(pts
+			(xy 119.38 81.28) (xy 139.7 81.28)
+		)
+		(stroke
+			(width 0)
+			(type default)
+		)
+	)
+	(wire
+		(pts
 			(xy 81.28 54.61) (xy 83.82 54.61)
 		)
@@
 		(pts
 			(xy 106.68 39.37) (xy 113.03 39.37)
+		)
+		(stroke
+			(width 0)
+			(type default)
+		)
+	)
+	(wire
+		(pts
+			(xy 119.38 88.9) (xy 139.7 88.9)
 		)
 		(stroke
@@
 			)
 			(justify left bottom)
+		)
+	)
+	(hierarchical_label "IMU_SDA"
+		(shape bidirectional)
+		(at 139.7 88.9 0)
+		(effects
+			(font
+				(size 1.27 1.27)
+			)
+			(justify left)
 		)
 	)
@@
 		)
 	)
+	(hierarchical_label "IMU_INT"
+		(shape input)
+		(at 139.7 83.82 0)
+		(effects
+			(font
+				(size 1.27 1.27)
+			)
+			(justify left)
+		)
+	)
+	(hierarchical_label "BURNWIRE_GATE"
+		(shape output)
+		(at 139.7 81.28 0)
+		(effects
+			(font
+				(size 1.27 1.27)
+			)
+			(justify left)
+		)
+	)
 	(hierarchical_label "RAIL_1_VOUT"
 		(shape input)
@@
 		)
 	)
+	(hierarchical_label "IMU_SCL"
+		(shape output)
+		(at 139.7 86.36 0)
+		(effects
+			(font
+				(size 1.27 1.27)
+			)
+			(justify left)
+		)
+	)

Commit message: finalize schematic
Parts:
- added J4: Conn_ARM_JTAG_SWD_10, Connector_PinHeader_1.27mm:PinHeader_2x05_P1.27mm_Vertical_SMD, symbol Connector:Conn_ARM_JTAG_SWD_10
- added R17: 10k, Resistor_SMD:R_0402_1005Metric, symbol Device:R_Small_US
Connections:
- net +3V3: now also J4.1 (VTref), R17.1; no longer U2.26 (RUN)
- net GND: now also J4.3 (GND), J4.5 (GND), J4.9 (GNDDetect)
- net SWCLK: now reaches U2.24 (SWCLK)
- net SWCLK: now also J4.4 (SWCLK/TCK)
- net SWDIO: now reaches U2.25 (SWDIO)
- net SWDIO: now also J4.2 (SWDIO/TMS)
- net ALERT: now reaches U2.6 (GPIO4)
- net GREEN_LED: now reaches U2.7 (GPIO5)
- net RED_LED: now reaches U2.8 (GPIO6)
- net IMU_SCL renamed SCL
- net IMU_SDA renamed SDA
- new net RESET: J4.10 (~{RESET}), R17.2, U2.26 (RUN)
- no-connect marks 16 -> 25
Other:
- note added: "SWD"
- moved on the sheet: C20, C21, C22, J3, R11, R8, R9, U3

Commit message: update footprint assignments and start layout
Parts:
- C20: footprint Capacitor_SMD:C_0603_1608Metric -> Capacitor_SMD:C_0402_1005Metric
- C23: footprint Capacitor_SMD:C_0402_1005Metric_Pad0.74x0.62mm_HandSolder -> Capacitor_SMD:C_0402_1005Metric
- C9: footprint Capacitor_SMD:C_0402_1005Metric -> Capacitor_SMD:C_0603_1608Metric
Changed lines of the file:
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@@
 			)
 		)
-		(property "Footprint" "Capacitor_SMD:C_0402_1005Metric"
+		(property "Footprint" "Capacitor_SMD:C_0603_1608Metric"
 			(at 116.84 58.42 0)
 			(hide yes)
@@
 			)
 		)
-		(property "Footprint" "Capacitor_SMD:C_0603_1608Metric"
+		(property "Footprint" "Capacitor_SMD:C_0402_1005Metric"
 			(at 260.35 71.12 0)
 			(hide yes)
@@
 			)
 		)
-		(property "Footprint" "Capacitor_SMD:C_0402_1005Metric_Pad0.74x0.62mm_HandSolder"
+		(property "Footprint" "Capacitor_SMD:C_0402_1005Metric"
 			(at 25.4 44.45 0)
 			(hide yes)

Commit message: start layout
Connections:
- net CAN_TX: now reaches U2.11 (GPIO8)
- net STB: now reaches U2.12 (GPIO9)
- net CAN_RX: now reaches U2.9 (GPIO7)
- no-connect marks 25 -> 22
Other:
- moved on the sheet: C13, C14, C15, C16, C17, C18, C23

Commit message: replace IMU and continue layout
Parts:
- added R12, R18: 4.7k, Resistor_SMD:R_0402_1005Metric, symbol Device:R_Small_US
Connections:
- net RAIL_1_VOUT is gone; now on net +3V3: C12.1, C13.1, C14.1, C15.1, C16.1, C17.1, C18.1, C23.1, U2.1 (IOVDD), U2.10 (IOVDD), U2.22 (IOVDD), U2.33 (IOVDD), U2.42 (IOVDD), U2.43 (ADC_AVDD), U2.44 (VREG_VIN), U2.48 (USB_VDD), U2.49 (IOVDD)
- net CAN_RX: now also U2.12 (GPIO9); no longer U2.9 (GPIO7)
- net IMU_INT: now also U2.5 (GPIO3); no longer U2.3 (GPIO1)
- net SCL: now also R18.2
- net SDA: now also U2.3 (GPIO1), R12.2; no longer U2.5 (GPIO3)
- net STB: now also U2.9 (GPIO7); no longer U2.12 (GPIO9)
- net MNT_INT: now reaches U2.13 (GPIO10)
- net SHUNT_SCL: now reaches U2.36 (GPIO24)
- net SHUNT_SDA: now reaches U2.37 (GPIO25)
- new net +1V8: R12.1, R18.1
- no-connect marks 22 -> 19
