File: shared/kicad/subsheets/usb_c/usb_c.kicad_pcb (KiCad board)
At the start: 4 copper layers, 12.6 x 17 mm, 9 parts, among them J1 USB_C_Receptacle_USB2.0_16P, U1 USBLC6-2P6

Commit message: fixes!!!
Parts:
- FB1: footprint Inductor_SMD:L_0603_1608Metric -> Inductor_SMD:L_0402_1005Metric
- moved FB1 0.86 mm to (148.3, 95.8)
Connections:
- net /usb_c/UNPROT_USB_D+ renamed /USB-C/UNPROT_USB_D+
- net /usb_c/UNPROT_USB_D- renamed /USB-C/UNPROT_USB_D-
- net /usb_c/USB_D+ renamed /USB-C/USB_D+
- net /usb_c/USB_D- renamed /USB-C/USB_D-
- net Net-(C2-Pad1) renamed /USB-C/PI
- net Net-(J1-CC1) renamed /USB-C/CC1
- net Net-(J1-CC2) renamed /USB-C/CC2
- net Net-(J1-SHIELD) renamed /USB-C/FB
Routing:
- net /USB-C/FB: track 20.4 -> 19.6 mm
