File: shared/kicad/subsheets/usb_c/usb_c_overvoltage.kicad_sch (KiCad schematic)
At the start: 9 parts, among them J1 USB_C_Receptacle_USB2.0_16P, U1 USBLC6-2P6

Commit message: fixes!!!
Parts:
- C1: value 100nF -> 100n; LCSC PN (none) -> C307331
- C2: LCSC PN (none) -> C15195
- FB1: footprint Inductor_SMD:L_0603_1608Metric -> Inductor_SMD:L_0402_1005Metric; LCSC PN C338244 -> C76891
- FB2: LCSC PN (none) -> C76891
- J1: LCSC PN (none) -> C2988369
- R1, R2: LCSC PN (none) -> C25905
- U1: LCSC PN (none) -> C2827693
Connections:
- net PI: now reaches C2.1, FB2.1, J1.A4 (VBUS), J1.A9 (VBUS), J1.B4 (VBUS), J1.B9 (VBUS)
- net CC1: now reaches J1.A5 (CC1), R1.1
- net CC2: now reaches J1.B5 (CC2), R2.1
- net FB: now reaches FB1.1, J1.SH (SHIELD)
Changed lines of the file:
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@@
-	)
-	(junction
-		(at 114.3 129.54)
-		(diameter 0)
-		(color 0 0 0 0)
 	)
 	(junction
@@
 	(wire
 		(pts
-			(xy 114.3 129.54) (xy 114.3 130.81)
+			(xy 114.3 121.92) (xy 114.3 130.81)
 		)
 		(stroke
@@
 	(wire
 		(pts
-			(xy 204.47 101.6) (xy 214.63 101.6)
-		)
-		(stroke
-			(width 0)
-			(type default)
-		)
-	)
-	(wire
-		(pts
-			(xy 204.47 99.06) (xy 214.63 99.06)
+			(xy 204.47 101.6) (xy 232.41 101.6)
 		)
 		(stroke
@@
 	(wire
 		(pts
-			(xy 128.27 128.27) (xy 128.27 129.54)
-		)
-		(stroke
-			(width 0)
-			(type default)
-		)
-	)
-	(wire
-		(pts
 			(xy 92.71 129.54) (xy 106.68 129.54)
 		)
@@
 	(wire
 		(pts
-			(xy 114.3 121.92) (xy 114.3 129.54)
-		)
-		(stroke
-			(width 0)
-			(type default)
-		)
-	)
-	(wire
-		(pts
 			(xy 205.74 86.36) (xy 205.74 87.63)
 		)
@@
 	(wire
 		(pts
-			(xy 114.3 129.54) (xy 128.27 129.54)
-		)
-		(stroke
-			(width 0)
-			(type default)
-		)
-	)
-	(wire
-		(pts
 			(xy 199.39 82.55) (xy 199.39 86.36)
 		)
@@
 	(wire
 		(pts
+			(xy 204.47 99.06) (xy 232.41 99.06)
+		)
+		(stroke
+			(width 0)
+			(type default)
+		)
+	)
+	(wire
+		(pts
 			(xy 160.02 83.82) (xy 160.02 87.63)
 		)
@@
 			(width 0)
 			(type default)
+		)
+	)
+	(label "FB"
+		(at 106.68 123.19 0)
+		(effects
+			(font
+				(size 1.27 1.27)
+				(thickness 0.1588)
+			)
+			(justify left bottom)
+		)
+	)
+	(label "PI"
+		(at 135.89 83.82 0)
+		(effects
+			(font
+				(size 1.27 1.27)
+				(thickness 0.1588)
+			)
+			(justify left bottom)
 		)
 	)
@@
 		)
 	)
+	(label "CC2"
+		(at 129.54 91.44 0)
+		(effects
+			(font
+				(size 1.27 1.27)
+				(thickness 0.1588)
+			)
+			(justify left bottom)
+		)
+	)
 	(label "UNPROT_USB_D-"
 		(at 132.08 99.06 0)
@@
 		)
 	)
-	(hierarchical_label "USB_D+"
-		(shape bidirectional)
-		(at 214.63 101.6 0)
+	(label "CC1"
+		(at 129.54 88.9 0)
 		(effects
 			(font
 				(size 1.27 1.27)
+				(thickness 0.1588)
+			)
+			(justify left bottom)
+		)
+	)
+	(hierarchical_label "USB_D+"
+		(shape bidirectional)
+		(at 232.41 101.6 0)
+		(effects
+			(font
+				(size 1.27 1.27)
 			)
 			(justify left)
@@
 	(hierarchical_label "USB_D-"
 		(shape bidirectional)
-		(at 214.63 99.06 0)
+		(at 232.41 99.06 0)
 		(effects
 			(font
@@
 		(property "Description" "Ferrite bead, small symbol"
 			(at 170.18 83.82 0)
+			(hide yes)
+			(show_name no)
+			(do_not_autoplace no)
+			(effects
+				(font
+					(size 1.27 1.27)
+				)
+			)
+		)
+		(property "LCSC PN" "C76891"
+			(at 170.18 83.82 90)
 			(hide yes)
 			(show_name no)
@@
 	)
 	(symbol
-		(lib_id "power:PWR_FLAG")
-		(at 128.27 128.27 0)
-		(unit 1)
-		(body_style 1)
-		(exclude_from_sim no)
-		(in_bom yes)
-		(on_board yes)
-		(in_pos_files yes)
-		(dnp no)
-		(fields_autoplaced yes)
-		(property "Reference" "#FLG02"
-			(at 128.27 126.365 0)
-			(hide yes)
-			(show_name no)
-			(do_not_autoplace no)
-			(effects
-				(font
-					(size 1.27 1.27)
-				)
-			)
-		)
-		(property "Value" "PWR_FLAG"
-			(at 128.27 123.19 0)
-			(show_name no)
-			(do_not_autoplace no)
-			(effects
-				(font
-					(size 1.27 1.27)
-				)
-			)
-		)
-		(property "Footprint" ""
-			(at 128.27 128.27 0)
-			(hide yes)
-			(show_name no)
-			(do_not_autoplace no)
-			(effects
-				(font
-					(size 1.27 1.27)
-				)
-			)
-		)
-		(property "Datasheet" ""
-			(at 128.27 128.27 0)
-			(hide yes)
-			(show_name no)
-			(do_not_autoplace no)
-			(effects
-				(font
-					(size 1.27 1.27)
-				)
-			)
-		)
-		(property "Description" "Special symbol for telling ERC where power comes from"
-			(at 128.27 128.27 0)
-			(hide yes)
-			(show_name no)
-			(do_not_autoplace no)
-			(effects
-				(font
-					(size 1.27 1.27)
-				)
-			)
-		)
-		(pin "1"
-		)
-		(instances
-			(project "usb_c"
-				(path "/d08425fa-3630-4aa4-87e5-628aacc30d11/93863b4a-ed7f-46af-bbb5-711ec713fa5e"
-					(reference "#FLG02")
-					(unit 1)
-				)
-			)
-		)
-	)
-	(symbol
 		(lib_id "power:GND")
 		(at 160.02 93.98 0)
@@
 		(dnp no)
 		(property "Reference" "U1"
-			(at 201.422 105.918 0)
-			(show_name no)
-			(do_not_autoplace no)
-			(effects
-				(font
-					(size 1.27 1.27)
-				)
-				(justify left)
+			(at 196.088 105.918 0)
+			(show_name no)
+			(do_not_autoplace no)
+			(effects
+				(font
+					(size 1.27 1.27)
+				)
+				(justify right)
 			)
 		)
 		(property "Value" "USBLC6-2P6"
-			(at 201.422 108.458 0)
-			(show_name no)
-			(do_not_autoplace no)
-			(effects
-				(font
-					(size 1.27 1.27)
-				)
-				(justify left)
+			(at 196.088 108.458 0)
+			(show_name no)
+			(do_not_autoplace no)
+			(effects
+				(font
+					(size 1.27 1.27)
+				)
+				(justify right)
 			)
 		)
@@
 		)
 		(property "Description" "Very low capacitance ESD protection diode, 2 data-line, SOT-666"
+			(at 199.39 99.06 0)
+			(hide yes)
+			(show_name no)
+			(do_not_autoplace no)
+			(effects
+				(font
+					(size 1.27 1.27)
+				)
+			)
+		)
+		(property "LCSC PN" "C2827693"
 			(at 199.39 99.06 0)
 			(hide yes)
@@
 		(property "Description" "Resistor, small US symbol"
 			(at 138.43 88.9 0)
+			(hide yes)
+			(show_name no)
+			(do_not_autoplace no)
+			(effects
+				(font
+					(size 1.27 1.27)
+				)
+			)
+		)
+		(property "LCSC PN" "C25905"
+			(at 138.43 88.9 90)
 			(hide yes)
 			(show_name no)
@@
 			)
 		)
+		(property "LCSC PN" "C25905"
+			(at 138.43 91.44 90)
+			(hide yes)
+			(show_name no)
+			(do_not_autoplace no)
+			(effects
+				(font
+					(size 1.27 1.27)
+				)
+			)
+		)
 		(pin "1"
 		)
@@
 			)
 		)
-		(property "Value" "100nF"
+		(property "Value" "100n"
 			(at 208.28 91.5669 0)
 			(show_name no)
@@
 		)
 		(property "Description" "capacitor, small US symbol"
+			(at 205.74 90.17 0)
+			(hide yes)
+			(show_name no)
+			(do_not_autoplace no)
+			(effects
+				(font
+					(size 1.27 1.27)
+				)
+			)
+		)
+		(property "LCSC PN" "C307331"
 			(at 205.74 90.17 0)
 			(hide yes)
@@
 			)
 		)
+		(property "LCSC PN" "C2988369"
+			(at 114.3 99.06 0)
+			(hide yes)
+			(show_name no)
+			(do_not_autoplace no)
+			(effects
+				(font
+					(size 1.27 1.27)
+				)
+			)
+		)
 		(pin "A12"
 		)
@@
 			)
 		)
-		(property "Footprint" "Inductor_SMD:L_0603_1608Metric"
+		(property "Footprint" "Inductor_SMD:L_0402_1005Metric"
 			(at 104.902 125.73 90)
 			(hide yes)
@@
 			)
 		)
-		(property "LCSC PN" "C338244"
+		(property "LCSC PN" "C76891"
 			(at 106.68 125.73 0)
 			(hide yes)
@@
 			(at 160.02 90.17 0)
 			(hide yes)
+			(show_name no)
+			(do_not_autoplace no)
+			(effects
+				(font
+					(size 1.27 1.27)
+				)
+			)
+		)
+		(property "LCSC PN" "C15195"
+			(at 160.02 90.17 0)
+			(hide yes)
