File: eps/v2/hardware/i2c_mux_efuse_ctrl.kicad_sch (KiCad schematic)
At the start: 29 parts, among them U1 TCA9548APWR

Commit message: Finish #173 mux and rebuild #178 as rail eFuse EN control
#173: Q1/Q2 gate pull-downs, test points on VSYS and both PGs, FET MPN/LCSC, R40-45 footprints to 0402, pin 6 ERC exclusion.

#178: replace the TCA9548A sheet with 8 FET EN/UVLO pull-downs and boot-default gate pulls (r1 on, r2-r8 off), drawn in the #173 style. Sheet pins added on the top level, calc images.

Add TPS25947 and AO3400A datasheets.
Parts:
- removed C1: 100n, Capacitor_SMD:C_0603_1608Metric, symbol Device:C_Small_US
- removed R1, R10, R11, R12, R13, R14, R15, R16, R17, R18, R19, R2, R4, R5, R6, R7, R8, R9: 4.7k, Resistor_SMD:R_0603_1608Metric, symbol Device:R_Small_US
- removed R20, R21, R22, R23, R24, R25, R26, R27: 100k, Resistor_SMD:R_0603_1608Metric, symbol Device:R_Small_US
- removed R3: 10k, Resistor_SMD:R_0603_1608Metric, symbol Device:R_Small_US
- removed U1: TCA9548APWR, Package_SO:TSSOP-24_4.4x7.8mm_P0.65mm, symbol Interface_Expansion:TCA9548APWR
- added Q10, Q3, Q4, Q5, Q6, Q7, Q8, Q9: AO3400A, Package_TO_SOT_SMD:SOT-23, symbol Transistor_FET:AO3400A
- added R48, R49, R50, R51, R52, R53, R54, R55: 100k, Resistor_SMD:R_0402_1005Metric, symbol Device:R_Small_US
Connections:
- net +3V3: now also R49.1, R50.1, R51.1, R52.1, R53.1, R54.1, R55.1
- net GND: now also Q10.2 (S), Q3.2 (S), Q4.2 (S), Q5.2 (S), Q6.2 (S), Q7.2 (S), Q8.2 (S), Q9.2 (S), R48.2
- new net R1_EN: Q3.1 (G), R48.1
- new net R1_EN_UVLO: Q3.3 (D)
- new net R2_EN: Q4.1 (G), R49.2
- new net R2_EN_UVLO: Q4.3 (D)
- new net R3_EN: Q5.1 (G), R50.2
- new net R3_EN_UVLO: Q5.3 (D)
- new net R4_EN: Q6.1 (G), R51.2
- new net R4_EN_UVLO: Q6.3 (D)
- new net R5_EN: Q7.1 (G), R52.2
- new net R5_EN_UVLO: Q7.3 (D)
- new net R6_EN: Q8.1 (G), R53.2
- new net R6_EN_UVLO: Q8.3 (D)
- new net R7_EN: Q9.1 (G), R54.2
- new net R7_EN_UVLO: Q9.3 (D)
- new net R8_EN: Q10.1 (G), R55.2
- new net R8_EN_UVLO: Q10.3 (D)
Other:
- note added: "Boot Default Calculation"
- note added: "EN/UVLO Shutdown Calculation"
- note added: "Gate Drive Calculation"
- note added: "MCU high turns the FET on, which pulls the rail eFuse EN/UVLO low and turns the rail off. Each rail's EN/UVLO divider is on the power rail eFuse sheet (#176)."
- note added: "OSUSat"
- note added: "PWR_FLAG until the +3V3 source (#174) is drawn"
- note added: "Pull Resistor Current Calculation"
- note added: "The MCU pins float during reset, so the 100k on each gate sets the boot state: pull-down = rail on, pull-up to +3V3 = rail off."
- note added: "off at boot"
- note added: "on at boot"
- note added: "r1 Enable (OBC, 3.3 V)"
- note added: "r2 Enable (3.3 V)"
- note added: "r3 Enable (3.3 V)"
- note added: "r4 Enable (3.3 V)"
- note added: "r5 Enable (5 V)"
- note added: "r6 Enable (VSYS)"
- note added: "r7 Enable (TBD)"
- note added: "r8 Enable (TBD)"
- note removed: "Assumptions to confirm: - r1 is the OBC rail (v1 rail index 0). - These pulls could live on the rail eFuse sheet (#176) instead. - If #176 puts a UVLO divider on each eFuse EN pin, these values need to change."
- note removed: "Channel map (one channel per software rail, from the EPS V2 block diagram): CH0 r1 eFuse (in: 3.3 V) CH4 r5 eFuse (in: 5 V) CH1 r2 eFuse (in: 3.3 V) CH5 r6 eFuse (in: Unreg) CH2 r3 eFuse (in: 3.3 V) CH6 r7 eFuse (in: TBD) CH3 r4 eFuse (in: 3.3 V) CH7 r8 eFuse (in: TBD) The 8 rail eFuses are the same part, so their I2C addresses would collide on one bus. Downstream devices must not use 0x70 (the m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"
- note removed: "Channel pull-ups (each channel is its own bus and needs its own pull-ups)"
- note removed: "I2C MUX FOR eFuse TELEMETRY / CONTROL (TCA9548A, address 0x70)"
- note removed: "RAIL ENABLE BOOT DEFAULTS"
- note removed: "The MCU drives en x8 directly (block diagram). Its pins float during reset, so these set the boot state: r1 (OBC) pulled ON, r2-r8 pulled OFF (EPS boot flow, subsystem_info.md)."
- note removed: "Upstream pull-ups: drop these if the MCU sheet already has them."
- title: I2C Mux & eFuse Control -> Rail eFuse Enable Control
