File: adcs/v2/adcs_hardware/1V8 Rail.kicad_sch (KiCad schematic)
At the start: 3 parts, among them U1 AP2112K-1.2

Commit message: add SWD port
Connections:
- net 1V8 Rail renamed 1V8 out
Changed lines of the file:
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@@
 		)
 	)
-	(hierarchical_label "1V8 Rail"
+	(hierarchical_label "1V8 out"
 		(shape output)
 		(at 152.4 90.17 0)
