File: adcs/v2/adcs_hardware/STSPIN Current Driver.kicad_sch (KiCad schematic)
At the start: 5 parts, among them U5 STSPIN220

Commit message: organized main sheet, switched current drivers
Parts:
- removed U5: STSPIN220, Package_DFN_QFN:VQFN-16-1EP_3x3mm_P0.5mm_EP1.8x1.8mm, symbol Driver_Motor:STSPIN220
- added C24: 22n, symbol Device:C_US
- added U4: STSPIN240, Package_DFN_QFN:VQFN-16-1EP_3x3mm_P0.5mm_EP1.8x1.8mm, symbol Driver_Motor:STSPIN240
Connections:
- net 5V _Filtered: now also U4.6 (VS)
- net GND: now also C24.2, U4.7 (GND); no longer R_sense2.2
- net PWM: now also R_sense2.2; no longer R_sense2.1
- net at R_OFF2.1, R_RCOFF2.1: now also U4.12 (TOFF)
- new net: C24.1, R_sense2.1, U4.11 (REF)
Other:
- note added: "Average coil current (where D = duty cycle): I_coil = D * V_supply / R_coil"
- note added: "Choose PWM frequency at well above 1/(2pi*T) -- where T = L/R time constant of the coil"
