File: adcs/v1/1v8_ldo.kicad_sch (KiCad schematic)
At the start: 3 parts, among them U1 AP2112K-1.2

Commit message: wire pwm pins on motor drivers, clean up sheet
Changed lines of the file:
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@@
 	(paper "A4")
+	(junction
+		(at 146.05 97.79)
+		(diameter 0)
+		(color 0 0 0 0)
+	)
 	(junction
 		(at 125.73 97.79)
@@
 	(wire
 		(pts
-			(xy 143.51 97.79) (xy 149.86 97.79)
+			(xy 143.51 97.79) (xy 146.05 97.79)
 		)
 		(stroke
@@
 	(wire
 		(pts
-			(xy 152.4 97.79) (xy 152.4 96.52)
+			(xy 152.4 97.79) (xy 152.4 93.98)
 		)
 		(stroke
@@
 	(wire
 		(pts
+			(xy 146.05 93.98) (xy 146.05 97.79)
+		)
+		(stroke
+			(width 0)
+			(type default)
+		)
+	)
+	(wire
+		(pts
 			(xy 149.86 110.49) (xy 149.86 114.3)
 		)
@@
 		(pts
 			(xy 135.89 107.95) (xy 135.89 118.11)
+		)
+		(stroke
+			(width 0)
+			(type default)
+		)
+	)
+	(wire
+		(pts
+			(xy 146.05 97.79) (xy 149.86 97.79)
 		)
 		(stroke
@@
 	(symbol
 		(lib_id "power:+1V8")
-		(at 152.4 96.52 0)
+		(at 152.4 93.98 0)
 		(unit 1)
 		(body_style 1)
@@
 		(in_pos_files yes)
 		(dnp no)
-		(fields_autoplaced yes)
 		(property "Reference" "#PWR039"
-			(at 152.4 100.33 0)
+			(at 152.4 97.79 0)
 			(hide yes)
 			(show_name no)
@@
 		)
 		(property "Value" "+1V8"
-			(at 152.4 91.44 0)
+			(at 152.908 89.916 0)
 			(show_name no)
 			(do_not_autoplace no)
@@
 		)
 		(property "Footprint" ""
-			(at 152.4 96.52 0)
+			(at 152.4 93.98 0)
 			(hide yes)
 			(show_name no)
@@
 		)
 		(property "Datasheet" ""
-			(at 152.4 96.52 0)
+			(at 152.4 93.98 0)
 			(hide yes)
 			(show_name no)
@@
 		)
 		(property "Description" "Power symbol creates a global label with name \"+1V8\""
-			(at 152.4 96.52 0)
+			(at 152.4 93.98 0)
 			(hide yes)
 			(show_name no)
@@
 					(unit 1)
 				)
+			)
+		)
+	)
+	(symbol
+		(lib_id "power:PWR_FLAG")
+		(at 146.05 93.98 0)
+		(unit 1)
+		(body_style 1)
+		(exclude_from_sim no)
+		(in_bom yes)
+		(on_board yes)
+		(in_pos_files yes)
+		(dnp no)
+		(property "Reference" "#FLG04"
+			(at 146.05 92.075 0)
+			(hide yes)
+			(show_name no)
+			(do_not_autoplace no)
+			(effects
+				(font
+					(size 1.27 1.27)
+				)
+			)
+		)
+		(property "Value" "PWR_FLAG"
+			(at 144.78 89.916 0)
+			(show_name no)
+			(do_not_autoplace no)
+			(effects
+				(font
+					(size 1.27 1.27)
+				)
+			)
+		)
+		(property "Footprint" "Package_SO:TSSOP-28_4.4x9.7mm_P0.65mm"
+			(at 146.05 93.98 0)
+			(hide yes)
+			(show_name no)
+			(do_not_autoplace no)
+			(effects
+				(font
+					(size 1.27 1.27)
+				)
+			)
+		)
+		(property "Datasheet" ""
+			(at 146.05 93.98 0)
+			(hide yes)
+			(show_name no)
+			(do_not_autoplace no)
+			(effects
+				(font
+					(size 1.27 1.27)
+				)
+			)
+		)
+		(property "Description" "Special symbol for telling ERC where power comes from"
+			(at 146.05 93.98 0)
+			(hide yes)
+			(show_name no)
+			(do_not_autoplace no)
+			(effects
+				(font
+					(size 1.27 1.27)
+				)
+			)
+		)
+		(pin "1"
+		)
+		(instances
+			(project "adcs"
+				(path "/d4fa1041-51e8-429a-8be3-f1e5a35c2607/c3745443-cfeb-4998-b62c-1903e2db139a"
+					(reference "#FLG04")
+					(unit 1)
+				)
