File: adcs/v1/adcs.kicad_sch (KiCad schematic)
At the start: 15 parts, among them SW1 SW_Push, U2 STM32L4Q5CGTx

Commit message: wire pwm pins on motor drivers, clean up sheet
Other:
- sheet STSPIN Current Driver ports: added EN, PHA1, PHB1, PWMA1, PWMB1; removed none
- sheet STSPIN Current Driver1 ports: added EN, PHA2, PHB2, PWMA2, PWMB2; removed none
- sheet STSPIN Current Driver2 ports: added EN, PHA3, PHB3, PWMA3, PWMB3; removed none
- sheet USB-C ports: added USB_D+, USB_D-; removed none
- note added: "Inter-Board Connector"
- note added: "Magnetorquer Driver & Peripherals"
- note removed: "Magnetorquer Driver Peripherals"

Commit message: add IMU, begin wiring
Other:
- removed sheet STSPIN Current Driver
- added sheet IMU (IMU.kicad_sch)
- added sheet STSPIN Current Driver3 (current_driver.kicad_sch)
- sheet STSPIN Current Driver1 ports: added PHA1, PHB1, PWMA1, PWMB1; removed PHA2, PHB2, PWMA2, PWMB2
- sheet STSPIN Current Driver2 ports: added PHA2, PHB2, PWMA2, PWMB2; removed PHA3, PHB3, PWMA3, PWMB3
Changed lines of the file:
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@@
 	(rectangle
 		(start 152.4 45.72)
-		(end 262.89 163.83)
+		(end 287.02 163.83)
 		(stroke
 			(width 0)
@@
 	(wire
 		(pts
-			(xy 238.76 120.65) (xy 243.84 120.65)
+			(xy 232.41 115.57) (xy 237.49 115.57)
 		)
 		(stroke
@@
 	(wire
 		(pts
-			(xy 234.95 77.47) (xy 238.76 77.47)
+			(xy 228.6 72.39) (xy 232.41 72.39)
 		)
 		(stroke
@@
 	(wire
 		(pts
-			(xy 243.84 115.57) (xy 238.76 115.57)
+			(xy 237.49 110.49) (xy 232.41 110.49)
 		)
 		(stroke
@@
 	(wire
 		(pts
-			(xy 243.84 125.73) (xy 238.76 125.73)
+			(xy 237.49 120.65) (xy 232.41 120.65)
 		)
 		(stroke
@@
 	(wire
 		(pts
-			(xy 238.76 123.19) (xy 243.84 123.19)
+			(xy 232.41 118.11) (xy 237.49 118.11)
 		)
 		(stroke
@@
 	(wire
 		(pts
-			(xy 234.95 73.66) (xy 238.76 73.66)
+			(xy 228.6 68.58) (xy 232.41 68.58)
 		)
 		(stroke
@@
 	(wire
 		(pts
-			(xy 234.95 69.85) (xy 238.76 69.85)
+			(xy 228.6 64.77) (xy 232.41 64.77)
 		)
 		(stroke
@@
 	(wire
 		(pts
-			(xy 238.76 118.11) (xy 243.84 118.11)
+			(xy 232.41 113.03) (xy 237.49 113.03)
 		)
 		(stroke
@@
 	)
 	(label "3V3_RAIL_6"
-		(at 243.84 120.65 0)
+		(at 237.49 115.57 0)
 		(effects
 			(font
@@
 	)
 	(label "SWCLK"
-		(at 243.84 115.57 0)
+		(at 237.49 110.49 0)
 		(effects
 			(font
@@
 	)
 	(label "I2C1_SCL"
-		(at 238.76 69.85 0)
+		(at 232.41 64.77 0)
 		(effects
 			(font
@@
 	)
 	(label "MNT_INT"
-		(at 238.76 77.47 0)
+		(at 232.41 72.39 0)
 		(effects
 			(font
@@
 	)
 	(label "nRST"
-		(at 243.84 118.11 0)
+		(at 237.49 113.03 0)
 		(effects
 			(font
@@
 	)
 	(label "SWO"
-		(at 243.84 125.73 0)
+		(at 237.49 120.65 0)
 		(effects
 			(font
@@
 	)
 	(label "I2C1_SDA"
-		(at 238.76 73.66 0)
+		(at 232.41 68.58 0)
 		(effects
 			(font
@@
 	)
 	(label "SWDIO"
-		(at 243.84 123.19 0)
+		(at 237.49 118.11 0)
 		(effects
 			(font
@@
 	)
 	(sheet
-		(at 220.98 67.31)
+		(at 214.63 62.23)
 		(size 13.97 21.59)
 		(exclude_from_sim no)
@@
 		)
 		(property "Sheetname" "Magnetometer"
-			(at 220.98 66.5984 0)
+			(at 214.63 61.5184 0)
 			(show_name no)
 			(do_not_autoplace no)
@@
 		)
 		(property "Sheetfile" "magnetometer.kicad_sch"
-			(at 220.98 89.4846 0)
+			(at 214.63 84.4046 0)
 			(show_name no)
 			(do_not_autoplace no)
@@
 		)
 		(pin "SCL" input
-			(at 234.95 69.85 0)
+			(at 228.6 64.77 0)
 			(effects
 				(font
@@
 		)
 		(pin "SDA" bidirectional
-			(at 234.95 73.66 0)
+			(at 228.6 68.58 0)
 			(effects
 				(font
@@
 		)
 		(pin "MNT_INT" output
-			(at 234.95 77.47 0)
+			(at 228.6 72.39 0)
 			(effects
 				(font
@@
 			(color 0 0 0 0)
 		)
-		(property "Sheetname" "STSPIN Current Driver2"
+		(property "Sheetname" "STSPIN Current Driver3"
 			(at 170.18 127.5584 0)
 			(show_name no)
@@
 	)
 	(sheet
-		(at 220.98 113.03)
+		(at 214.63 107.95)
 		(size 17.78 16.51)
 		(exclude_from_sim no)
@@
 		)
 		(property "Sheetname" "SWD Connector"
-			(at 220.98 112.3184 0)
+			(at 214.63 107.2384 0)
 			(show_name no)
 			(do_not_autoplace no)
@@
 		)
 		(property "Sheetfile" "swd.kicad_sch"
-			(at 220.98 130.1246 0)
+			(at 214.63 125.0446 0)
 			(show_name no)
 			(do_not_autoplace no)
@@
 		)
 		(pin "3V3_IN" input
-			(at 238.76 120.65 0)
+			(at 232.41 115.57 0)
 			(effects
 				(font
@@
 		)
 		(pin "SWDIO" bidirectional
-			(at 238.76 123.19 0)
+			(at 232.41 118.11 0)
 			(effects
 				(font
@@
 		)
 		(pin "SWO" input
-			(at 238.76 125.73 0)
+			(at 232.41 120.65 0)
 			(effects
 				(font
@@
 		)
 		(pin "SWCLK" output
-			(at 238.76 115.57 0)
+			(at 232.41 110.49 0)
 			(effects
 				(font
@@
 		)
 		(pin "nRST" output
-			(at 238.76 118.11 0)
+			(at 232.41 113.03 0)
 			(effects
 				(font
@@
 			(color 0 0 0 0)
 		)
-		(property "Sheetname" "STSPIN Current Driver"
+		(property "Sheetname" "STSPIN Current Driver1"
 			(at 170.18 60.2484 0)
 			(show_name no)
@@
 			(color 0 0 0 0)
 		)
-		(property "Sheetname" "STSPIN Current Driver1"
+		(property "Sheetname" "STSPIN Current Driver2"
 			(at 170.18 94.5384 0)
 			(show_name no)
@@
 	)
 	(sheet
-		(at 220.98 95.25)
+		(at 214.63 90.17)
 		(size 13.97 10.16)
 		(exclude_from_sim no)
@@
 		)
 		(property "Sheetname" "1V8 Rail"
-			(at 220.98 94.5384 0)
+			(at 214.63 89.4584 0)
 			(show_name no)
 			(do_not_autoplace no)
@@
 		)
 		(property "Sheetfile" "1v8_ldo.kicad_sch"
-			(at 220.98 105.9946 0)
+			(at 214.63 100.9146 0)
 			(show_name no)
 			(do_not_autoplace no)
@@
 	)
 	(sheet
-		(at 220.98 135.89)
+		(at 214.63 130.81)
 		(size 15.24 12.7)
 		(exclude_from_sim no)
@@
 		)
 		(property "Sheetname" "USB-C"
-			(at 220.98 135.1784 0)
+			(at 214.63 130.0984 0)
 			(show_name no)
 			(do_not_autoplace no)
@@
 		)
 		(property "Sheetfile" "usb_c.kicad_sch"
-			(at 220.98 149.1746 0)
+			(at 214.63 144.0946 0)
 			(show_name no)
 			(do_not_autoplace no)
@@
 		)
 		(pin "USB_D+" bidirectional
-			(at 236.22 138.43 0)
+			(at 229.87 133.35 0)
 			(effects
 				(font
@@
 		)
 		(pin "USB_D-" bidirectional
-			(at 236.22 140.97 0)
+			(at 229.87 135.89 0)
 			(effects
 				(font
@@
 				)
 			)
+		)
+	)
+	(sheet
+		(at 255.27 62.23)
+		(size 15.24 17.78)
+		(exclude_from_sim no)
+		(in_bom yes)
+		(on_board yes)
+		(dnp no)
+		(fields_autoplaced yes)
+		(stroke
+			(width 0.1524)
+			(type solid)
+		)
+		(fill
+			(color 0 0 0 0)
+		)
+		(property "Sheetname" "IMU"
+			(at 255.27 61.5184 0)
+			(show_name no)
+			(do_not_autoplace no)
+			(effects
+				(font
+					(size 1.27 1.27)
+				)
+				(justify left bottom)
+			)
+		)
+		(property "Sheetfile" "IMU.kicad_sch"
+			(at 255.27 80.5946 0)
+			(show_name no)
+			(do_not_autoplace no)
+			(effects
+				(font
+					(size 1.27 1.27)
+				)
+				(justify left top)
+			)
+		)
+		(instances
+			(project "adcs"
+				(path "/d4fa1041-51e8-429a-8be3-f1e5a35c2607"
+					(page "10")
+				)
+			)

Commit message: swap STSPIN240 for the STSPIN250 current driver, begin wiring
Other:
- sheet STSPIN Current Driver1 ports: added PH1, PWM1; removed PHA1, PHB1, PWMA1, PWMB1
- sheet STSPIN Current Driver2 ports: added PH1, PWM1; removed PHA2, PHB2, PWMA2, PWMB2
- sheet STSPIN Current Driver3 ports: added PH1, PWM1; removed PHA3, PHB3, PWMA3, PWMB3
Changed lines of the file:
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@@
 			)
 		)
-		(pin "PHA3" input
+		(pin "PH1" input
 			(at 170.18 138.43 180)
 			(effects
@@
 			)
 		)
-		(pin "PHB3" input
+		(pin "PWM1" input
 			(at 170.18 140.97 180)
-			(effects
-				(font
-					(size 1.27 1.27)
-				)
-				(justify left)
-			)
-		)
-		(pin "PWMA3" input
-			(at 170.18 143.51 180)
-			(effects
-				(font
-					(size 1.27 1.27)
-				)
-				(justify left)
-			)
-		)
-		(pin "PWMB3" input
-			(at 170.18 146.05 180)
 			(effects
 				(font
@@
 			)
 		)
-		(pin "PHA1" input
+		(pin "PH1" input
 			(at 170.18 69.85 180)
 			(effects
@@
 			)
 		)
-		(pin "PHB1" input
+		(pin "PWM1" input
 			(at 170.18 72.39 180)
-			(effects
-				(font
-					(size 1.27 1.27)
-				)
-				(justify left)
-			)
-		)
-		(pin "PWMA1" input
-			(at 170.18 74.93 180)
-			(effects
-				(font
-					(size 1.27 1.27)
-				)
-				(justify left)
-			)
-		)
-		(pin "PWMB1" input
-			(at 170.18 77.47 180)
 			(effects
 				(font
@@
 			)
 		)
-		(pin "PHA2" input
+		(pin "PH1" input
 			(at 170.18 105.41 180)
 			(effects
@@
 			)
 		)
-		(pin "PHB2" input
+		(pin "PWM1" input
 			(at 170.18 107.95 180)
 			(effects
 				(font
-					(size 1.27 1.27)
-				)
-				(justify left)
-			)
-		)
-		(pin "PWMA2" input
-			(at 170.18 110.49 180)
-			(effects
-				(font
-					(size 1.27 1.27)
-				)
-				(justify left)
-			)
-		)
-		(pin "PWMB2" input
-			(at 170.18 113.03 180)
-			(effects
-				(font

Commit message: finish wiring for STSPIN250s, still need to connect to MCU
Connections:
- net USBC-D-: now reaches U2.22 (PB11)
- net USBC-D+: now reaches U2.25 (PB12)
- no-connect marks 34 -> 32
Other:
- sheet IMU ports: added IMU_SCL, IMU_SDA; removed none
- sheet STSPIN Current Driver1 ports: added PH; removed PH1, PWM1
- sheet STSPIN Current Driver2 ports: added PH; removed PH1, PWM1
- sheet STSPIN Current Driver3 ports: added PH; removed PH1, PWM1
